File: wifi-board/wifi-board.sch (KiCad schematic (older format))
At the start: 13 parts, among them J1 UFL, J2 UFL, J49 SBBJ49, J50 SBBJ50, U1 ap6356s, Y1 37.4MHz, 1.6x1.2mm, Epson FA-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

Commit message: update
Connections:
- net labels added: BT_UART_CTS, BT_UART_RTS, BT_UART_TX
- wire segments 91 -> 94
Changed lines of the file:
@@
 	2300 3850 3350 3850
 Wire Wire Line
-	4850 5850 7800 5850
-Wire Wire Line
-	4850 5950 7800 5950
-Wire Wire Line
-	4850 6050 7800 6050
+	7050 5950 7800 5950
 Wire Wire Line
 	3350 6250 2750 6250
@@
 Wire Wire Line
 	4850 5750 5700 5750
-Text Label 5150 5750 0    60   ~ 0
-BT_UART_RX
 Wire Wire Line
 	7800 5750 7050 5750
 Text Label 7050 5750 0    60   ~ 0
-BT_UART_RX
+BT_UART_TX
 Text Notes 5800 2550 0    60   ~ 0
 crystal oscillator, 37.4MHz recommended.\nsee cypress cyw4356 datasheet.
@@
 Text Notes 10350 3050 0    60   ~ 0
 ELL4GG4R7N
+Wire Wire Line
+	7800 5850 7050 5850
+Text Label 7050 5850 0    60   ~ 0
+BT_UART_RX
+Wire Wire Line
+	4850 5850 5700 5850
+Text Label 5150 5850 0    60   ~ 0
+BT_UART_TX
+Text Label 5150 5750 0    60   ~ 0
+BT_UART_RX
+Text Label 7050 5950 0    60   ~ 0
+BT_UART_RTS
+Wire Wire Line
+	7800 6050 7050 6050
+Text Label 7050 6050 0    60   ~ 0
+BT_UART_CTS
+Wire Wire Line
+	4850 5950 5700 5950
+Text Label 5150 5950 0    60   ~ 0
+BT_UART_CTS
+Wire Wire Line
+	4850 6050 5700 6050
+Text Label 5150 6050 0    60   ~ 0
+BT_UART_RTS
 $EndSCHEMATC
